Commit message: updating engrais_gazebo package

File: engrais_gazebo/models/plantgreen/plantgreen.xacro (robot description, xacro)
@@ -1,4 +1,5 @@
 <?xml version="1.0" ?>
 <sdf version="1.5" xmlns:xacro="http://www.ros.org/wiki/xacro">
+    <!-- macro to compute the inertia of the cylinder -->
     <xacro:macro name="cylinder_inertia" params="m r h">
         <inertia>
@@ -8,11 +9,15 @@
         </inertia>
     </xacro:macro>
-    <xacro:property name="body_mass"   value="0.100" /> <!-- arbitrary value for mass -->
-    <xacro:property name="body_radius" value="0.100" /> <!-- Square dimensions (widthxwidth) of beams -->
-    <xacro:property name="body_length" value="0.010" /> <!-- Square dimensions (widthxwidth) of beams -->
-    <xacro:property name="stem_mass"   value="0.010" /> <!-- arbitrary value for mass -->
-    <xacro:property name="stem_radius" value="0.050" /> <!-- Square dimensions (widthxwidth) of beams -->
-    <xacro:property name="stem_length" value="1.000" /> <!-- Square dimensions (widthxwidth) of beams -->
+    <!-- constants -->
+    <!-- the body constants (body = base = a kind of root), use to make the plant more stabled -->
+    <xacro:property name="body_mass"   value="0.100" /> <!-- mass of the body - kg -->
+    <xacro:property name="body_radius" value="0.100" /> <!-- radius of the body - m -->
+    <xacro:property name="body_length" value="0.010" /> <!-- length of the body - m -->
+    <!-- the stem constant -->
+    <xacro:property name="stem_mass"   value="0.010" /> <!-- mass of the stem - kg -->
+    <xacro:property name="stem_radius" value="0.050" /> <!-- radius of the stem - m -->
+    <xacro:property name="stem_length" value="1.000" /> <!-- length of the stem - m -->
     <model name="plantgreen">
+        <!-- the body of the plant -->
         <link name="body">
             <pose>0 0 ${body_length/2} 0 0 0</pose>
@@ -36,4 +41,5 @@
                     </cylinder>
                 </geometry>
+                <!-- we want the green plant to be green... -->
                 <material>
                     <ambient>0.1 0.5 0.1 1</ambient>
@@ -44,4 +50,5 @@
             </visual>
         </link>
+        <!-- the stem of the plant -->
         <link name="stem">
             <pose>0 0 ${body_length+stem_length/2+0.001} 0 0 0</pose>
@@ -73,4 +80,5 @@
             </visual>
         </link>
+       <!-- fixed joint between the stem and the body, as it is not possible to define a fixed joint, we define a revolute joint with no limits -->
        <joint name="body_stem_joint" type="revolute">
           <parent>body</parent>

File: engrais_gazebo/models/plantred/plantred.xacro (robot description, xacro)
@@ -1,4 +1,5 @@
 <?xml version="1.0" ?>
 <sdf version="1.5" xmlns:xacro="http://www.ros.org/wiki/xacro">
+    <!-- macro to compute the inertia of the cylinder -->
     <xacro:macro name="cylinder_inertia" params="m r h">
         <inertia>
@@ -8,11 +9,15 @@
         </inertia>
     </xacro:macro>
-    <xacro:property name="body_mass"   value="0.500" /> <!-- arbitrary value for mass -->
-    <xacro:property name="body_radius" value="0.100" /> <!-- Square dimensions (widthxwidth) of beams -->
-    <xacro:property name="body_length" value="0.010" /> <!-- Square dimensions (widthxwidth) of beams -->
-    <xacro:property name="stem_mass"   value="0.010" /> <!-- arbitrary value for mass -->
-    <xacro:property name="stem_radius" value="0.050" /> <!-- Square dimensions (widthxwidth) of beams -->
-    <xacro:property name="stem_length" value="1.000" /> <!-- Square dimensions (widthxwidth) of beams -->
+    <!-- constants -->
+    <!-- the body constants (body = base = a kind of root), use to make the plant more stabled -->
+    <xacro:property name="body_mass"   value="0.500" /> <!-- mass of the body - kg -->
+    <xacro:property name="body_radius" value="0.100" /> <!-- radius of the body - m -->
+    <xacro:property name="body_length" value="0.010" /> <!-- length of the body - m -->
+    <!-- the stem constant -->
+    <xacro:property name="stem_mass"   value="0.010" /> <!-- mass of the stem - kg -->
+    <xacro:property name="stem_radius" value="0.050" /> <!-- radius of the stem - m -->
+    <xacro:property name="stem_length" value="1.000" /> <!-- length of the stem - m -->
     <model name="plantred">
+        <!-- the body of the plant -->
         <link name="body">
             <pose>0 0 ${body_length/2} 0 0 0</pose>
@@ -36,4 +41,5 @@
                     </cylinder>
                 </geometry>
+                <!-- we want the red plant to be red... -->
                 <material>
                     <ambient>0.5 0.1 0.1 1</ambient>
@@ -44,4 +50,5 @@
             </visual>
         </link>
+        <!-- the stem of the plant -->
         <link name="stem">
             <pose>0 0 ${body_length+stem_length/2+0.001} 0 0 0</pose>
@@ -73,4 +80,5 @@
             </visual>
         </link>
+       <!-- fixed joint between the stem and the body, as it is not possible to define a fixed joint, we define a revolute joint with no limits -->
        <joint name="body_stem_joint" type="revolute">
           <parent>body</parent>

File: engrais_gazebo/worlds/engrais.world.xacro (robot description, xacro)
@@ -1,10 +1,11 @@
 <?xml version="1.0" ?>
 <sdf version="1.5" xmlns:xacro="http://www.ros.org/wiki/xacro">
-    <!-- We use a custom world for the rrbot so that the camera angle is launched correctly -->
-    <xacro:property name="nb_rows"              value="4"    /> <!-- arbitrary value for mass -->
-    <xacro:property name="nb_plants_row"        value="30"   /> <!-- Square dimensions (widthxwidth) of beams -->
-    <xacro:property name="space_between_rows"   value="3.00" /> <!-- Square dimensions (widthxwidth) of beams -->
-    <xacro:property name="space_between_plants" value="0.30" /> <!-- Square dimensions (widthxwidth) of beams -->
+    <!-- default simple world using population grid tag -->
+    <xacro:property name="nb_rows"              value="4"    /> <!-- number of rows in the field -->
+    <xacro:property name="nb_plants_row"        value="30"   /> <!-- number of plants in a row -->
+    <xacro:property name="space_between_rows"   value="3.00" /> <!-- space between the rows -->
+    <xacro:property name="space_between_plants" value="0.30" /> <!-- space between the plants in a row -->
     <world name="default">
+        <!-- standard plane -->
         <include>
             <uri>model://ground_plane</uri>
@@ -28,18 +29,4 @@
             </distribution>
         </population>
-        <!-- <population name="vegetablesRED">
-        <model name="plantred">
-        <include>
-        <uri>model://plantred</uri>
-        </include>
-        </model>
-        <pose>12 5 0 0 0 0</pose>
-        <distribution>
-        <type>grid</type>
-        <rows>40</rows>
-        <cols>1</cols>
-        <step>3 0.25 0</step>
-        </distribution>
-        </population> -->
     </world>
 </sdf>
