Commit message: cleaning the engrais_description package

File: engrais_description/urdf/engrais.xacro (robot description, xacro)
@@ -1,35 +1,41 @@
 <?xml version="1.0"?>
-<!-- Revolute-Revolute Manipulator -->
+<!--Engrais robot description -->
 <robot name="engrais" xmlns:xacro="http://www.ros.org/wiki/xacro">
-  <!-- Constants for robot dimensions -->
-    <xacro:property name="PI" value="3.1415926535897931"/>
-    <xacro:property name="body_mass"     value="10"  /> <!-- arbitrary value for mass -->
-    <xacro:property name="body_width_x"  value="$(arg body_size_x)"   /> <!-- Square dimensions (widthxwidth) of beams -->
-    <xacro:property name="body_width_y"  value="1"   /> <!-- Square dimensions (widthxwidth) of beams -->
-    <xacro:property name="body_height"   value="0.5" /> <!-- Square dimensions (widthxwidth) of beams -->
-    <xacro:property name="caster_radius" value="0.15"/> <!-- arbitrary value for mass -->
-    <xacro:property name="caster_mass"   value="0.1"/>  <!-- arbitrary value for mass -->
-    <xacro:property name="wheel_mass"   value="1"    /> <!-- arbitrary value for mass -->
-    <xacro:property name="wheel_radius" value="0.3" /> <!-- Square dimensions (widthxwidth) of beams -->
-    <xacro:property name="wheel_length"    value="0.2" /> <!-- Square dimensions (widthxwidth) of beams -->
-    <xacro:property name="sick_size"      value="0.1" /> <!-- Square dimensions (widthxwidth) of beams -->
-    <xacro:property name="sick_range_max" value="4.0" /> <!-- Square dimensions (widthxwidth) of beams -->
-    <xacro:property name="sick_range_min" value="0.1" /> <!-- Square dimensions (widthxwidth) of beams -->
-    <xacro:property name="sick_nb_msr"    value="360" /> <!-- Square dimensions (widthxwidth) of beams -->
-    <xacro:property name="sick_min_angle" value="${-PI/2}" /> <!-- Square dimensions (widthxwidth) of beams -->
-    <xacro:property name="sick_max_angle" value="${PI/2}" /> <!-- Square dimensions (widthxwidth) of beams -->
-    <!-- Import all Gazebo-customization elements, including Gazebo colors -->
+    <!--  Constants -->
+    <xacro:property name="PI" value="3.1415926535897931"/> <!-- PI value -->
+    <!--  Constants for the robot body -->
+    <xacro:property name="body_mass"     value="10"  />                <!-- body mass - kg -->
+    <xacro:property name="body_width_x"  value="$(arg body_size_x)" /> <!-- body lenght - m -->
+    <xacro:property name="body_width_y"  value="1"   />                <!-- body width - m -->
+    <xacro:property name="body_height"   value="0.5" />                <!-- body height - m -->
+    <!--  Constants for the caster wheels, front and back -->
+    <xacro:property name="caster_radius" value="0.15"/> <!-- radius of the caster wheel - m -->
+    <xacro:property name="caster_mass"   value="0.1"/>  <!-- mass of the caster wheel - m -->
+    <!--  Constants for the differentials wheels, left and right -->
+    <xacro:property name="wheel_mass"   value="1"   />    <!-- wheel mass - kg -->
+    <xacro:property name="wheel_radius" value="0.3" />    <!-- wheel radius - m -->
+    <xacro:property name="wheel_length"    value="0.2" /> <!-- wheel length -->
+    <!--  Constants for the LiDAR -->
+    <xacro:property name="sick_size"      value="0.1" />      <!-- The LiDAR is represented by a box with sick_size size - m -->
+    <xacro:property name="sick_range_max" value="4.0" />      <!-- Maximal range for the LiDAR - m -->
+    <xacro:property name="sick_range_min" value="0.1" />      <!-- Minimal range for the LiDAR - m -->
+    <xacro:property name="sick_nb_msr"    value="360" />      <!-- Number of measurements in one data set -->
+    <xacro:property name="sick_min_angle" value="${-PI/2}" /> <!-- Minimal angle range -->
+    <xacro:property name="sick_max_angle" value="${PI/2}" />  <!-- Maximal angle range -->
+    <!-- Import all Gazebo-customization elements, including Gazebo colors, LiDAR plugins... -->
     <xacro:include filename="$(find engrais_description)/urdf/engrais.gazebo" />
     <!-- Import Rviz colors -->
     <xacro:include filename="$(find engrais_description)/urdf/materials.xacro" />
-    <!-- Import Rviz colors -->
+    <!-- Import some macro the clean the code -->
     <xacro:include filename="$(find engrais_description)/urdf/macros.xacro" />
     <!--    ****************** LINKS ****************** -->
+    <!-- artificial base link -->
     <link name="footprint" />
+    <!-- Fixed joint between the artificial based link and the body -->
     <joint name="base_joint" type="fixed">
         <parent link="footprint"/>
         <child link="body"/>
     </joint>
-    <!-- Base Link -->
+    <!-- Body Link -->
     <link name="body">
         <collision name="body_collision">
@@ -52,5 +58,5 @@
         </inertial>
     </link>
-    <!-- caster wheel Link -->
+    <!-- Back caster wheel Link -->
     <link name="caster_wheel_back">
         <collision>
@@ -73,4 +79,5 @@
         </inertial>
     </link>
+    <!-- fixed joint between the back caster wheel and the body -->
     <joint name="joint_body_caster_wheel_back" type="fixed">
         <parent link="body"/>
@@ -78,5 +85,5 @@
         <origin xyz="${-body_width_x/2+caster_radius} 0 ${-body_height/2}" rpy="0 0 0"/>
     </joint>
-    <!-- caster wheel Link -->
+    <!-- Front caster wheel Link -->
     <link name="caster_wheel_front">
         <collision>
@@ -99,4 +106,5 @@
         </inertial>
     </link>
+    <!-- fixed joint between the front caster wheel and the body -->
     <joint name="joint_body_caster_wheel_front" type="fixed">
         <parent link="body"/>
@@ -104,4 +112,5 @@
         <origin xyz="${body_width_x/2-caster_radius} 0 ${-body_height/2}" rpy="0 0 0"/>
     </joint>
+    <!-- Front LiDAR Link -->
     <link name="sick_front_link">
         <visual>
@@ -113,4 +122,5 @@
         </visual>
     </link>
+    <!-- fixed joint between the front LiDAR and the body -->
     <joint name="sick_front_joint" type="fixed">
         <origin xyz="${body_width_x/2 - sick_size/2} 0 ${body_height/2+sick_size/2}" rpy="0 0 0" />
@@ -118,4 +128,5 @@
         <child link="sick_front_link" />
     </joint>
+    <!-- Back LiDAR Link -->
     <link name="sick_back_link">
         <visual>
@@ -127,4 +138,5 @@
         </visual>
     </link>
+    <!-- fixed joint between the back LiDAR and the body -->
     <joint name="sick_back_joint" type="fixed">
         <origin xyz="-${body_width_x/2 - sick_size/2} 0 ${body_height/2+sick_size/2}" rpy="0 0 ${PI}" />
@@ -132,7 +144,6 @@
         <child link="sick_back_link" />
     </joint>
-<!-- ******************** WHEELS LINK ******************** -->
+    <!-- macros are used to set the wheel links and joints -->
     <wheel leftright="right" parent="body" translateX="0" translateY="${-body_width_y/2-wheel_length/2}" translateZ="${-body_height/2+(wheel_radius-caster_radius)}" wheel_mass="${wheel_mass}" wheel_radius="${wheel_radius}" wheel_height="${wheel_length}"/>
     <wheel leftright="left" parent="body" translateX="0" translateY="${body_width_y/2+wheel_length/2}" translateZ="${-body_height/2+(wheel_radius-caster_radius)}" wheel_mass="${wheel_mass}" wheel_radius="${wheel_radius}" wheel_height="${wheel_length}"/>
-    <!--    ****************** JOINTS ****************** -->
 </robot>

File: engrais_description/urdf/macros.xacro (robot description, xacro)
@@ -1,4 +1,7 @@
 <?xml version="1.0"?>
+<!-- macros used to clean the code -->
 <robot xmlns:xacro="http://www.ros.org/wiki/xacro">
+    <!-- macros to compute classical inertia matrices -->
+    <!-- inertia of a cylinder -->
     <xacro:macro name="cylinder_inertia" params="m r h">
         <inertia  ixx="${m*(3*r*r+h*h)/12}" ixy = "0" ixz = "0"
@@ -7,4 +10,5 @@
         />
     </xacro:macro>
+    <!-- inertia of a box -->
     <xacro:macro name="box_inertia" params="m x y z">
         <inertia  ixx="${m*(y*y+z*z)/12}" ixy = "0" ixz = "0"
@@ -13,4 +17,5 @@
         />
     </xacro:macro>
+    <!-- inertia of a sphere -->
     <xacro:macro name="sphere_inertia" params="m r">
         <inertia  ixx="${2*m*r*r/5}" ixy = "0" ixz = "0"
@@ -19,5 +24,7 @@
         />
     </xacro:macro>
+    <!-- macro use for the left and right wheels -->
     <xacro:macro name="wheel" params="leftright parent translateX translateY translateZ wheel_mass wheel_radius wheel_height">
+        <!-- defines the link of the wheel -->
         <link name="${leftright}_wheel">
             <visual>
@@ -40,4 +47,5 @@
             </inertial>
         </link>
+        <!-- defines the joint between the wheel and the body -->
         <joint name="${leftright}_wheel_joint" type="continuous">
             <parent link="${parent}"/>
@@ -59,4 +67,5 @@
             </actuator>
         </transmission>
+        <!-- gazebo informations for the wheel -->
         <gazebo reference="${leftright}_wheel">
             <mu1 value="10"/>

Commit message: gazebo model update

File: engrais_description/urdf/engrais.xacro (robot description, xacro)
@@ -55,5 +55,5 @@
             <origin xyz="0 0 0" rpy="0 0 0"/>
             <mass value="${body_mass}"/>
-            <box_inertia m="${body_mass}" x="${body_width_x}" y="${body_width_y}" z="${body_mass}"/>
+            <box_inertia m="${body_mass}" x="${body_width_x}" y="${body_width_y}" z="${body_height}"/>
         </inertial>
     </link>

File: engrais_description/urdf/macros.xacro (robot description, xacro)
@@ -5,21 +5,24 @@
     <!-- inertia of a cylinder -->
     <xacro:macro name="cylinder_inertia" params="m r h">
-        <inertia  ixx="${m*(3*r*r+h*h)/12}" ixy = "0" ixz = "0"
-            iyy="${m*(3*r*r+h*h)/12}" iyz = "0"
-            izz="${m*r*r/2}"
+        <inertia
+            ixx="${1/12.0 * m * (3*r*r + h*h)}" ixy = "0" ixz = "0"
+            iyy="${1/12.0 * m * (3*r*r + h*h)}" iyz = "0"
+            izz="${1/2.0 * m * r*r}"
         />
     </xacro:macro>
     <!-- inertia of a box -->
     <xacro:macro name="box_inertia" params="m x y z">
-        <inertia  ixx="${m*(y*y+z*z)/12}" ixy = "0" ixz = "0"
-            iyy="${m*(x*x+z*z)/12}" iyz = "0"
-            izz="${m*(x*x+z*z)/12}"
+        <inertia
+            ixx="${1/12.0 * m * (y*y + z*z)}" ixy = "0" ixz = "0"
+            iyy="${1/12.0 * m * (x*x + z*z)}" iyz = "0"
+            izz="${1/12.0 * m * (x*x + y*y)}"
         />
     </xacro:macro>
     <!-- inertia of a sphere -->
     <xacro:macro name="sphere_inertia" params="m r">
-        <inertia  ixx="${2*m*r*r/5}" ixy = "0" ixz = "0"
-            iyy="${2*m*r*r/5}" iyz = "0"
-            izz="${2*m*r*r/5}"
+        <inertia
+            ixx="${2.0/5.0 * m * r*r}" ixy = "0" ixz = "0"
+            iyy="${2.0/5.0 * m * r*r}" iyz = "0"
+            izz="${2.0/5.0 * m * r*r}"
         />
     </xacro:macro>
@@ -43,5 +46,5 @@
             <inertial>
                 <mass value="${wheel_mass}" />
-                <origin xyz="0 0 0" />
+                <origin xyz="0 0 0" rpy="${PI/2} 0 0 " />
                 <cylinder_inertia  m="${wheel_mass}" r="${wheel_radius}" h="${wheel_height}" />
             </inertial>

Commit message: changes made to select lines, gazebo simulation, launch files

File: engrais_description/urdf/engrais.xacro (robot description, xacro)
@@ -1,3 +1,3 @@
-<?xml version="1.0"?>
+<?xml version="1.6"?>
 <!--Engrais robot description -->
 <robot name="engrais" xmlns:xacro="http://www.ros.org/wiki/xacro">
@@ -7,13 +7,13 @@
     <xacro:property name="body_mass"     value="10"  />                <!-- body mass - kg -->
     <xacro:property name="body_width_x"  value="$(arg body_size_x)" /> <!-- body lenght - m -->
-    <xacro:property name="body_width_y"  value="1"   />                <!-- body width - m -->
-    <xacro:property name="body_height"   value="0.5" />                <!-- body height - m -->
+    <xacro:property name="body_width_y"  value="0.4"   />                <!-- body width - m -->
+    <xacro:property name="body_height"   value="0.2" />                <!-- body height - m -->
     <!--  Constants for the caster wheels, front and back -->
-    <xacro:property name="caster_radius" value="0.15"/> <!-- radius of the caster wheel - m -->
+    <xacro:property name="caster_radius" value="0.10"/> <!-- radius of the caster wheel - m -->
     <xacro:property name="caster_mass"   value="0.1"/>  <!-- mass of the caster wheel - m -->
     <!--  Constants for the differentials wheels, left and right -->
     <xacro:property name="wheel_mass"   value="1"   />    <!-- wheel mass - kg -->
-    <xacro:property name="wheel_radius" value="0.3" />    <!-- wheel radius - m -->
-    <xacro:property name="wheel_length"    value="0.2" /> <!-- wheel length -->
+    <xacro:property name="wheel_radius" value="0.22" />    <!-- wheel radius - m -->
+    <xacro:property name="wheel_length"    value="0.15" /> <!-- wheel length -->
     <!--  Constants for the LiDAR -->
     <xacro:property name="sick_size"      value="0.1" />      <!-- The LiDAR is represented by a box with sick_size size - m -->
@@ -31,5 +31,6 @@
     <!--    ****************** LINKS ****************** -->
     <!-- artificial base link -->
-    <link name="footprint" />
+    <link name="footprint">
+    </link>
     <!-- Fixed joint between the artificial based link and the body -->
     <joint name="base_joint" type="fixed">
@@ -90,5 +91,5 @@
             <origin xyz="0 0 0" rpy="0 0 0"/>
             <geometry>
-            <sphere radius="${caster_radius}"/>
+                <sphere radius="${caster_radius}"/>
             </geometry>
         </collision>

File: engrais_description/urdf/macros.xacro (robot description, xacro)
@@ -1,3 +1,3 @@
-<?xml version="1.0"?>
+<?xml version="1.6"?>
 <!-- macros used to clean the code -->
 <robot xmlns:xacro="http://www.ros.org/wiki/xacro">
@@ -46,5 +46,5 @@
             <inertial>
                 <mass value="${wheel_mass}" />
-                <origin xyz="0 0 0" rpy="${PI/2} 0 0 " />
+                <origin xyz="0 0 0" rpy="${PI/2} 0 0" />
                 <cylinder_inertia  m="${wheel_mass}" r="${wheel_radius}" h="${wheel_height}" />
             </inertial>
